Commit message: added GPU lidar simulation support and set it as default.

File: simulation/simulation_with_velodyne_in_gazebo9_ws/src/velodyne_simulator/velodyne_description/urdf/HDL-32E.urdf.xacro (robot description, xacro)
@@ -2,5 +2,5 @@
 <robot xmlns:xacro="http://www.ros.org/wiki/xacro" name="HDL-32E">
   <xacro:property name="M_PI" value="3.1415926535897931" />
-  <xacro:macro name="HDL-32E" params="parent name topic *origin">
+  <xacro:macro name="HDL-32E" params="*origin parent:=base_link name:=velodyne topic:=/velodyne_points hz:=10 lasers:=32 samples:=2187 collision_range:=0.3 min_range:=0.9 max_range:=130.0 noise:=0.008 min_angle:=-${M_PI} max_angle:=${M_PI} gpu:=false">
     <joint name="${name}_base_mount_joint" type="fixed">
       <xacro:insert_block name="origin" />
@@ -10,7 +10,9 @@
     <link name="${name}_base_link">
       <inertial>
-        <mass value="0.1"/>
-        <origin xyz="0 0 0"/>
-        <inertia ixx="0.1" ixy="0" ixz="0" iyy="0.1" iyz="0" izz="0.1"/>
+        <mass value="1.0"/>
+        <origin xyz="0 0 0.07212"/>
+        <inertia ixx="${(1.0 * (3.0*0.04267*0.04267 + 0.14424*0.14424)) / 12.0}" ixy="0" ixz="0"
+          iyy="${(1.0 * (3.0*0.04267*0.04267 + 0.14424*0.14424)) / 12.0}" iyz="0"
+          izz="${0.5 * 1.0 * (0.04267*0.04267)}"/>
       </inertial>
       <visual>
@@ -33,7 +35,7 @@
     <link name="${name}">
       <inertial>
-        <mass value="0.1"/>
+        <mass value="0.01"/>
         <origin xyz="0 0 0"/>
-        <inertia ixx="0.1" ixy="0" ixz="0" iyy="0.1" iyz="0" izz="0.1"/>
+        <inertia ixx="1e-7" ixy="0" ixz="0" iyy="1e-7" iyz="0" izz="1e-7"/>
       </inertial>
       <visual>
@@ -46,42 +48,84 @@
     <!-- Gazebo requires the velodyne_gazebo_plugins package -->
     <gazebo reference="${name}">
-      <sensor type="ray" name="${name}-HDL32E">
-        <pose>0 0 0 0 0 0</pose>
-        <visualize>false</visualize>
-        <update_rate>10</update_rate>
-        <ray>
-          <scan>
-            <horizontal>
-              <samples>2187</samples> <!-- Change this to 500 if gazebo keeps timing out -->
-              <resolution>1</resolution>
-              <min_angle>-${M_PI}</min_angle>
-              <max_angle> ${M_PI}</max_angle>
-            </horizontal>
-            <vertical>
-              <samples>32</samples>
-              <resolution>1</resolution>
-              <min_angle>-${30.67*M_PI/180.0}</min_angle>
-              <max_angle> ${10.67*M_PI/180.0}</max_angle>
-            </vertical>
-          </scan>
-          <range>
-            <min>0.055</min>
-            <max>140.0</max>
-            <resolution>0.001</resolution>
-          </range>
-          <noise>
-            <type>gaussian</type>
-            <mean>0.0</mean>
-            <stddev>0.0</stddev>
-          </noise>
-        </ray>
-        <plugin name="gazebo_ros_laser_controller" filename="libgazebo_ros_velodyne_laser.so">
-          <topicName>${topic}</topicName>
-          <frameName>/${name}</frameName>
-          <min_range>0.9</min_range>
-          <max_range>130.0</max_range>
-          <gaussianNoise>0.008</gaussianNoise>
-        </plugin>
-      </sensor>
+      <xacro:if value="${gpu}">
+        <sensor type="gpu_ray" name="${name}-HDL32E">
+          <pose>0 0 0 0 0 0</pose>
+          <visualize>false</visualize>
+          <update_rate>${hz}</update_rate>
+          <ray>
+            <scan>
+              <horizontal>
+                <samples>${samples}</samples>
+                <resolution>1</resolution>
+                <min_angle>${min_angle}</min_angle>
+                <max_angle>${max_angle}</max_angle>
+              </horizontal>
+              <vertical>
+                <samples>${lasers}</samples>
+                <resolution>1</resolution>
+                <min_angle>-${30.67*M_PI/180.0}</min_angle>
+                <max_angle> ${10.67*M_PI/180.0}</max_angle>
+              </vertical>
+            </scan>
+            <range>
+              <min>${collision_range}</min>
+              <max>${max_range+1}</max>
+              <resolution>0.001</resolution>
+            </range>
+            <noise>
+              <type>gaussian</type>
+              <mean>0.0</mean>
+              <stddev>0.0</stddev>
+            </noise>
+          </ray>
+          <plugin name="gazebo_ros_laser_controller" filename="libgazebo_ros_velodyne_gpu_laser.so">
+            <topicName>${topic}</topicName>
+            <frameName>${name}</frameName>
+            <min_range>${min_range}</min_range>
+            <max_range>${max_range}</max_range>
+            <gaussianNoise>${noise}</gaussianNoise>
+          </plugin>
+        </sensor>
+      </xacro:if>
+      <xacro:unless value="${gpu}">
+        <sensor type="ray" name="${name}-HDL32E">
+          <pose>0 0 0 0 0 0</pose>
+          <visualize>false</visualize>
+          <update_rate>${hz}</update_rate>
+          <ray>
+            <scan>
+              <horizontal>
+                <samples>${samples}</samples>
+                <resolution>1</resolution>
+                <min_angle>${min_angle}</min_angle>
+                <max_angle>${max_angle}</max_angle>
+              </horizontal>
+              <vertical>
+                <samples>${lasers}</samples>
+                <resolution>1</resolution>
+                <min_angle>-${30.67*M_PI/180.0}</min_angle>
+                <max_angle> ${10.67*M_PI/180.0}</max_angle>
+              </vertical>
+            </scan>
+            <range>
+              <min>${collision_range}</min>
+              <max>${max_range+1}</max>
+              <resolution>0.001</resolution>
+            </range>
+            <noise>
+              <type>gaussian</type>
+              <mean>0.0</mean>
+              <stddev>0.0</stddev>
+            </noise>
+          </ray>
+          <plugin name="gazebo_ros_laser_controller" filename="libgazebo_ros_velodyne_laser.so">
+            <topicName>${topic}</topicName>
+            <frameName>${name}</frameName>
+            <min_range>${min_range}</min_range>
+            <max_range>${max_range}</max_range>
+            <gaussianNoise>${noise}</gaussianNoise>
+          </plugin>
+        </sensor>
+      </xacro:unless>
     </gazebo>
   </xacro:macro>

File: simulation/simulation_with_velodyne_in_gazebo9_ws/src/velodyne_simulator/velodyne_description/urdf/VU-8.urdf-rotating.xacro (robot description, xacro)
@@ -1,6 +1,15 @@
 <?xml version="1.0"?>
-<robot xmlns:xacro="http://www.ros.org/wiki/xacro" name="VLP-16">
+<robot xmlns:xacro="http://www.ros.org/wiki/xacro" name="VU-8">
   <xacro:property name="M_PI" value="3.1415926535897931" />
-  <xacro:macro name="VLP-16" params="*origin parent:=base_link name:=velodyne topic:=/velodyne_points hz:=10 lasers:=16 samples:=1875 collision_range:=0.3 min_range:=0.9 max_range:=130.0 noise:=0.008 min_angle:=-${M_PI} max_angle:=${M_PI} gpu:=false">
+  <!-- Minimum horizontal angle is -100 DEG - Wide FOV -->
+  <xacro:property name="min_horizontal_angle" value="-3.14159" />
+  <!-- Maximum horizontal angle is 100 DEG - Wide FOV -->
+  <xacro:property name="max_horizontal_angle" value="3.14159" />
+  <!-- Minimum vertical angle is -3 DEG -->
+  <xacro:property name="min_vertical_angle" value="-0.523599" />
+  <!-- Maximum vertical angle is 3 DEG-->
+  <xacro:property name="max_vertical_angle" value="0.523599" />
+  <xacro:macro name="VU-8" params="
+    *origin parent:=base_link name:=leddar topic:=/leddar_points hz:=10 lasers:=8 samples:=1875 collision_range:=0.3 min_range:=0.1 max_range:=130.0 noise:=0.008 gpu:=false">
     <joint name="${name}_base_mount_joint" type="fixed">
       <xacro:insert_block name="origin" />
@@ -10,9 +19,7 @@
     <link name="${name}_base_link">
       <inertial>
-        <mass value="0.83"/>
+        <mass value="1e-2"/>
         <origin xyz="0 0 0.03585"/>
-        <inertia ixx="${(0.83 * (3.0*0.0516*0.0516 + 0.0717*0.0717)) / 12.0}" ixy="0" ixz="0"
-          iyy="${(0.83 * (3.0*0.0516*0.0516 + 0.0717*0.0717)) / 12.0}" iyz="0"
-          izz="${0.5 * 0.83 * (0.0516*0.0516)}"/>
+        <inertia ixx="1e-2" ixy="0" ixz="0" iyy="1e-2" iyz="0" izz="1e-2"/>
       </inertial>
       <visual>
@@ -33,14 +40,9 @@
       </collision>
     </link>
-    <joint name="${name}_base_scan_joint" type="fixed" >
-      <origin xyz="0 0 0.0377" rpy="0 0 0" />
-      <parent link="${name}_base_link" />
-      <child link="${name}"/>
-    </joint>
-    <link name="${name}">
+    <link name="rotating_${name}">
       <inertial>
-        <mass value="0.01"/>
+        <mass value="1e-2"/>
         <origin xyz="0 0 0"/>
-        <inertia ixx="1e-7" ixy="0" ixz="0" iyy="1e-7" iyz="0" izz="1e-7"/>
+        <inertia ixx="1e-2" ixy="0" ixz="0" iyy="1e-2" iyz="0" izz="1e-2"/>
       </inertial>
       <visual>
@@ -51,8 +53,24 @@
       </visual>
     </link>
+    <joint name="${name}_base_scan_joint" type="revolute" >
+      <origin xyz="0 0 0.0377" rpy="0 0 0" />
+      <parent link="${name}_base_link" />
+      <child link="rotating_${name}"/>
+      <limit effort="10.0" lower="-0.5" upper="0.5" velocity="0.1"/>
+      <axis xyz="0 0 1" />
+    </joint>
+    <transmission name="simple_trans">
+      <type>transmission_interface/SimpleTransmission</type>
+      <joint name="${name}_base_scan_joint">
+        <hardwareInterface>hardware_interface/EffortJointInterface</hardwareInterface>
+      </joint>
+      <actuator name="foo_motor">
+        <hardwareInterface>hardware_interface/EffortJointInterface</hardwareInterface>
+      </actuator>
+    </transmission>
     <!-- Gazebo requires the velodyne_gazebo_plugins package -->
-    <gazebo reference="${name}">
+    <gazebo reference="rotating_${name}">
       <xacro:if value="${gpu}">
-        <sensor type="gpu_ray" name="${name}-VLP16">
+        <sensor type="gpu_ray" name="${name}-VU8">
           <pose>0 0 0 0 0 0</pose>
           <visualize>false</visualize>
@@ -63,12 +81,12 @@
                 <samples>${samples}</samples>
                 <resolution>1</resolution>
-                <min_angle>${min_angle}</min_angle>
-                <max_angle>${max_angle}</max_angle>
+                <min_angle>${min_horizontal_angle}</min_angle>
+                <max_angle>${max_horizontal_angle}</max_angle>
               </horizontal>
               <vertical>
                 <samples>${lasers}</samples>
                 <resolution>1</resolution>
-                <min_angle>-${15.0*M_PI/180.0}</min_angle>
-                <max_angle> ${15.0*M_PI/180.0}</max_angle>
+                <min_angle>${min_vertical_angle}</min_angle>
+                <max_angle>${max_vertical_angle}</max_angle>
               </vertical>
             </scan>
@@ -86,13 +104,15 @@
           <plugin name="gazebo_ros_laser_controller" filename="libgazebo_ros_velodyne_gpu_laser.so">
             <topicName>${topic}</topicName>
-            <frameName>${name}</frameName>
+            <frameName>rotating_${name}</frameName>
             <min_range>${min_range}</min_range>
             <max_range>${max_range}</max_range>
             <gaussianNoise>${noise}</gaussianNoise>
+            <staticFrameName>${name}_base_link</staticFrameName>
+            <staticTopicName>${topic}_static</staticTopicName>
           </plugin>
         </sensor>
       </xacro:if>
       <xacro:unless value="${gpu}">
-        <sensor type="ray" name="${name}-VLP16">
+        <sensor type="ray" name="${name}-VU8">
           <pose>0 0 0 0 0 0</pose>
           <visualize>false</visualize>
@@ -103,12 +123,12 @@
                 <samples>${samples}</samples>
                 <resolution>1</resolution>
-                <min_angle>${min_angle}</min_angle>
-                <max_angle>${max_angle}</max_angle>
+                <min_angle>${min_horizontal_angle}</min_angle>
+                <max_angle>${max_horizontal_angle}</max_angle>
               </horizontal>
               <vertical>
                 <samples>${lasers}</samples>
                 <resolution>1</resolution>
-                <min_angle>-${15.0*M_PI/180.0}</min_angle>
-                <max_angle> ${15.0*M_PI/180.0}</max_angle>
+                <min_angle>${min_vertical_angle}</min_angle>
+                <max_angle>${max_vertical_angle}</max_angle>
               </vertical>
             </scan>
@@ -126,8 +146,10 @@
           <plugin name="gazebo_ros_laser_controller" filename="libgazebo_ros_velodyne_laser.so">
             <topicName>${topic}</topicName>
-            <frameName>${name}</frameName>
+            <frameName>rotating_${name}</frameName>
             <min_range>${min_range}</min_range>
             <max_range>${max_range}</max_range>
             <gaussianNoise>${noise}</gaussianNoise>
+            <staticFrameName>${name}_base_link</staticFrameName>
+            <staticTopicName>${topic}_static</staticTopicName>
           </plugin>
         </sensor>

File: simulation/simulation_with_velodyne_in_gazebo9_ws/src/velodyne_simulator/velodyne_description/urdf/VU-8.urdf.xacro (robot description, xacro)
@@ -1,6 +1,15 @@
 <?xml version="1.0"?>
-<robot xmlns:xacro="http://www.ros.org/wiki/xacro" name="VLP-16">
+<robot xmlns:xacro="http://www.ros.org/wiki/xacro" name="VU-8">
   <xacro:property name="M_PI" value="3.1415926535897931" />
-  <xacro:macro name="VLP-16" params="*origin parent:=base_link name:=velodyne topic:=/velodyne_points hz:=10 lasers:=16 samples:=1875 collision_range:=0.3 min_range:=0.9 max_range:=130.0 noise:=0.008 min_angle:=-${M_PI} max_angle:=${M_PI} gpu:=false">
+  <!-- Minimum horizontal angle is -100 DEG - Wide FOV -->
+  <xacro:property name="min_horizontal_angle" value="-3.14159" />
+  <!-- Maximum horizontal angle is 100 DEG - Wide FOV -->
+  <xacro:property name="max_horizontal_angle" value="3.14159" />
+  <!-- Minimum vertical angle is -3 DEG -->
+  <xacro:property name="min_vertical_angle" value="-0.523599" />
+  <!-- Maximum vertical angle is 3 DEG-->
+  <xacro:property name="max_vertical_angle" value="0.523599" />
+  <xacro:macro name="VU-8" params="
+    *origin parent:=base_link name:=leddar topic:=/leddar_points hz:=10 lasers:=8 samples:=1875 collision_range:=0.3 min_range:=0.1 max_range:=130.0 noise:=0.008 gpu:=false">
     <joint name="${name}_base_mount_joint" type="fixed">
       <xacro:insert_block name="origin" />
@@ -10,9 +19,7 @@
     <link name="${name}_base_link">
       <inertial>
-        <mass value="0.83"/>
+        <mass value="1e-7"/>
         <origin xyz="0 0 0.03585"/>
-        <inertia ixx="${(0.83 * (3.0*0.0516*0.0516 + 0.0717*0.0717)) / 12.0}" ixy="0" ixz="0"
-          iyy="${(0.83 * (3.0*0.0516*0.0516 + 0.0717*0.0717)) / 12.0}" iyz="0"
-          izz="${0.5 * 0.83 * (0.0516*0.0516)}"/>
+        <inertia ixx="1e-7" ixy="0" ixz="0" iyy="1e-7" iyz="0" izz="1e-7"/>
       </inertial>
       <visual>
@@ -40,5 +47,5 @@
     <link name="${name}">
       <inertial>
-        <mass value="0.01"/>
+        <mass value="1e-7"/>
         <origin xyz="0 0 0"/>
         <inertia ixx="1e-7" ixy="0" ixz="0" iyy="1e-7" iyz="0" izz="1e-7"/>
@@ -54,5 +61,5 @@
     <gazebo reference="${name}">
       <xacro:if value="${gpu}">
-        <sensor type="gpu_ray" name="${name}-VLP16">
+        <sensor type="gpu_ray" name="${name}-VU8">
           <pose>0 0 0 0 0 0</pose>
           <visualize>false</visualize>
@@ -63,12 +70,12 @@
                 <samples>${samples}</samples>
                 <resolution>1</resolution>
-                <min_angle>${min_angle}</min_angle>
-                <max_angle>${max_angle}</max_angle>
+                <min_angle>${min_horizontal_angle}</min_angle>
+                <max_angle>${max_horizontal_angle}</max_angle>
               </horizontal>
               <vertical>
                 <samples>${lasers}</samples>
                 <resolution>1</resolution>
-                <min_angle>-${15.0*M_PI/180.0}</min_angle>
-                <max_angle> ${15.0*M_PI/180.0}</max_angle>
+                <min_angle>${min_vertical_angle}</min_angle>
+                <max_angle>${max_vertical_angle}</max_angle>
               </vertical>
             </scan>
@@ -94,5 +101,5 @@
       </xacro:if>
       <xacro:unless value="${gpu}">
-        <sensor type="ray" name="${name}-VLP16">
+        <sensor type="ray" name="${name}-VU8">
           <pose>0 0 0 0 0 0</pose>
           <visualize>false</visualize>
@@ -103,12 +110,12 @@
                 <samples>${samples}</samples>
                 <resolution>1</resolution>
-                <min_angle>${min_angle}</min_angle>
-                <max_angle>${max_angle}</max_angle>
+                <min_angle>${min_horizontal_angle}</min_angle>
+                <max_angle>${max_horizontal_angle}</max_angle>
               </horizontal>
               <vertical>
                 <samples>${lasers}</samples>
                 <resolution>1</resolution>
-                <min_angle>-${15.0*M_PI/180.0}</min_angle>
-                <max_angle> ${15.0*M_PI/180.0}</max_angle>
+                <min_angle>${min_vertical_angle}</min_angle>
+                <max_angle>${max_vertical_angle}</max_angle>
               </vertical>
             </scan>

File: simulation/simulation_with_velodyne_in_gazebo9_ws/src/velodyne_simulator/velodyne_description/urdf/example.urdf.xacro (robot description, xacro)
@@ -1,4 +1,6 @@
 <?xml version="1.0"?>
 <robot xmlns:xacro="http://www.ros.org/wiki/xacro" name="example">
+  <xacro:arg name="gpu" default="false"/>
+  <xacro:property name="gpu" value="$(arg gpu)" />
   <!-- Base Footprint -->
   <link name="base_footprint" />
@@ -29,9 +31,9 @@
   </link>
   <xacro:include filename="$(find velodyne_description)/urdf/VLP-16.urdf.xacro"/>
-  <VLP-16 parent="base_link" name="velodyne" topic="/velodyne_points">
+  <VLP-16 parent="base_link" name="velodyne" topic="/velodyne_points" hz="10" samples="440" gpu="${gpu}">
     <origin xyz="0 0 0.4" rpy="0 0 0" />
   </VLP-16>
   <xacro:include filename="$(find velodyne_description)/urdf/HDL-32E.urdf.xacro"/>
-  <HDL-32E parent="base_link" name="velodyne2" topic="/velodyne_points2">
+  <HDL-32E parent="base_link" name="velodyne2" topic="/velodyne_points2" hz="10" samples="220" gpu="${gpu}">
     <origin xyz="0 0 0.6" rpy="0 0 0" />
   </HDL-32E>

File: simulation/simulation_with_velodyne_in_gazebo9_ws/src/velodyne_simulator/velodyne_simulator/velodyne_description/urdf/VU-8.urdf.xacro (robot description, xacro)
@@ -1,6 +1,15 @@
 <?xml version="1.0"?>
-<robot xmlns:xacro="http://www.ros.org/wiki/xacro" name="VLP-16">
+<robot xmlns:xacro="http://www.ros.org/wiki/xacro" name="VU-8">
   <xacro:property name="M_PI" value="3.1415926535897931" />
-  <xacro:macro name="VLP-16" params="*origin parent:=base_link name:=velodyne topic:=/velodyne_points hz:=10 lasers:=16 samples:=1875 collision_range:=0.3 min_range:=0.9 max_range:=130.0 noise:=0.008 min_angle:=-${M_PI} max_angle:=${M_PI} gpu:=false">
+  <!-- Minimum horizontal angle is -100 DEG - Wide FOV -->
+  <xacro:property name="min_horizontal_angle" value="-1.74533" />
+  <!-- Maximum horizontal angle is 100 DEG - Wide FOV -->
+  <xacro:property name="max_horizontal_angle" value="1.74533" />
+  <!-- Minimum vertical angle is -3 DEG -->
+  <xacro:property name="min_vertical_angle" value="-0.0523599" />
+  <!-- Maximum vertical angle is 3 DEG-->
+  <xacro:property name="max_vertical_angle" value="0.0523599" />
+  <xacro:macro name="VU-8" params="
+    *origin parent:=base_link name:=leddar topic:=/leddar_points hz:=10 lasers:=8 samples:=1875 collision_range:=0.3 min_range:=0.9 max_range:=130.0 noise:=0.008 gpu:=false">
     <joint name="${name}_base_mount_joint" type="fixed">
       <xacro:insert_block name="origin" />
@@ -10,9 +19,7 @@
     <link name="${name}_base_link">
       <inertial>
-        <mass value="0.83"/>
+        <mass value="1e-7"/>
         <origin xyz="0 0 0.03585"/>
-        <inertia ixx="${(0.83 * (3.0*0.0516*0.0516 + 0.0717*0.0717)) / 12.0}" ixy="0" ixz="0"
-          iyy="${(0.83 * (3.0*0.0516*0.0516 + 0.0717*0.0717)) / 12.0}" iyz="0"
-          izz="${0.5 * 0.83 * (0.0516*0.0516)}"/>
+        <inertia ixx="1e-7" ixy="0" ixz="0" iyy="1e-7" iyz="0" izz="1e-7"/>
       </inertial>
       <visual>
@@ -40,5 +47,5 @@
     <link name="${name}">
       <inertial>
-        <mass value="0.01"/>
+        <mass value="1e-7"/>
         <origin xyz="0 0 0"/>
         <inertia ixx="1e-7" ixy="0" ixz="0" iyy="1e-7" iyz="0" izz="1e-7"/>
@@ -54,5 +61,5 @@
     <gazebo reference="${name}">
       <xacro:if value="${gpu}">
-        <sensor type="gpu_ray" name="${name}-VLP16">
+        <sensor type="gpu_ray" name="${name}-VU8">
           <pose>0 0 0 0 0 0</pose>
           <visualize>false</visualize>
@@ -63,12 +70,12 @@
                 <samples>${samples}</samples>
                 <resolution>1</resolution>
-                <min_angle>${min_angle}</min_angle>
-                <max_angle>${max_angle}</max_angle>
+                <min_angle>${min_horizontal_angle}</min_angle>
+                <max_angle>${max_horizontal_angle}</max_angle>
               </horizontal>
               <vertical>
                 <samples>${lasers}</samples>
                 <resolution>1</resolution>
-                <min_angle>-${15.0*M_PI/180.0}</min_angle>
-                <max_angle> ${15.0*M_PI/180.0}</max_angle>
+                <min_angle>${min_vertical_angle}</min_angle>
+                <max_angle>${max_vertical_angle}</max_angle>
               </vertical>
             </scan>
@@ -94,5 +101,5 @@
       </xacro:if>
       <xacro:unless value="${gpu}">
-        <sensor type="ray" name="${name}-VLP16">
+        <sensor type="ray" name="${name}-VU8">
           <pose>0 0 0 0 0 0</pose>
           <visualize>false</visualize>
@@ -103,12 +110,12 @@
                 <samples>${samples}</samples>
                 <resolution>1</resolution>
-                <min_angle>${min_angle}</min_angle>
-                <max_angle>${max_angle}</max_angle>
+                <min_angle>${min_horizontal_angle}</min_angle>
+                <max_angle>${max_horizontal_angle}</max_angle>
               </horizontal>
               <vertical>
                 <samples>${lasers}</samples>
                 <resolution>1</resolution>
-                <min_angle>-${15.0*M_PI/180.0}</min_angle>
-                <max_angle> ${15.0*M_PI/180.0}</max_angle>
+                <min_angle>${min_vertical_angle}</min_angle>
+                <max_angle>${max_vertical_angle}</max_angle>
               </vertical>
             </scan>
